Commit message: add-bumi3_4340_point.urdf

File: gear_sonic/data/assets/robot_description/urdf/bumi3/bumi3_4340_point.urdf (robot description, URDF)
Before this commit: robot BUMI_V3.0_260119, 22 links, 21 joints
Links:
- link base_link: geometry visual mesh filename=../../meshes/bumi3/base_link.STL
- link l_ankle_pitch_link: geometry collision mesh filename=../../meshes/bumi3/l_ankle_pitch_link.STL; visual mesh filename=../../meshes/bumi3/l_ankle_pitch_link.STL
- link l_ankle_roll_link: geometry collision sphere radius=0.005; collision sphere radius=0.005
- link l_arm_pitch_link: geometry collision mesh filename=../../meshes/bumi3/l_arm_pitch_link.STL; visual mesh filename=../../meshes/bumi3/l_arm_pitch_link.STL
- link l_arm_roll_link: geometry collision mesh filename=../../meshes/bumi3/l_arm_roll_link.STL; visual mesh filename=../../meshes/bumi3/l_arm_roll_link.STL
- link l_arm_yaw_link: geometry collision mesh filename=../../meshes/bumi3/l_arm_yaw_link.STL; visual mesh filename=../../meshes/bumi3/l_arm_yaw_link.STL
- link l_elbow_pitch_link: geometry collision mesh filename=../../meshes/bumi3/l_elbow_pitch_link.STL scale=1.15 1.15 1.15; visual mesh filename=../../meshes/bumi3/l_elbow_pitch_link.STL
- link l_knee_pitch_link: geometry collision mesh filename=../../meshes/bumi3/l_knee_pitch_link.STL; visual mesh filename=../../meshes/bumi3/l_knee_pitch_link.STL
- link l_leg_pitch_link: geometry collision mesh filename=../../meshes/bumi3/l_leg_pitch_link.STL; visual mesh filename=../../meshes/bumi3/l_leg_pitch_link.STL
- link l_leg_roll_link: geometry collision mesh filename=../../meshes/bumi3/l_leg_roll_link.STL; visual mesh filename=../../meshes/bumi3/l_leg_roll_link.STL
- link l_leg_yaw_link: geometry collision mesh filename=../../meshes/bumi3/l_leg_yaw_link.STL; visual mesh filename=../../meshes/bumi3/l_leg_yaw_link.STL
- link r_ankle_pitch_link: geometry collision mesh filename=../../meshes/bumi3/r_ankle_pitch_link.STL; visual mesh filename=../../meshes/bumi3/r_ankle_pitch_link.STL
- link r_ankle_roll_link: geometry collision sphere radius=0.005; collision sphere radius=0.005
- link r_arm_pitch_link: geometry collision mesh filename=../../meshes/bumi3/r_arm_pitch_link.STL; visual mesh filename=../../meshes/bumi3/r_arm_pitch_link.STL
- link r_arm_roll_link: geometry collision mesh filename=../../meshes/bumi3/r_arm_roll_link.STL; visual mesh filename=../../meshes/bumi3/r_arm_roll_link.STL
- link r_arm_yaw_link: geometry collision mesh filename=../../meshes/bumi3/r_arm_yaw_link.STL; visual mesh filename=../../meshes/bumi3/r_arm_yaw_link.STL
- link r_elbow_pitch_link: geometry collision mesh filename=../../meshes/bumi3/r_elbow_pitch_link.STL scale=1.15 1.15 1.15; visual mesh filename=../../meshes/bumi3/r_elbow_pitch_link.STL
- link r_knee_pitch_link: geometry collision mesh filename=../../meshes/bumi3/r_knee_pitch_link.STL; visual mesh filename=../../meshes/bumi3/r_knee_pitch_link.STL
- link r_leg_pitch_link: geometry collision mesh filename=../../meshes/bumi3/r_leg_pitch_link.STL; visual mesh filename=../../meshes/bumi3/r_leg_pitch_link.STL
- link r_leg_roll_link: geometry collision mesh filename=../../meshes/bumi3/r_leg_roll_link.STL; visual mesh filename=../../meshes/bumi3/r_leg_roll_link.STL
- link r_leg_yaw_link: geometry collision mesh filename=../../meshes/bumi3/r_leg_yaw_link.STL; visual mesh filename=../../meshes/bumi3/r_leg_yaw_link.STL
- link waist_yaw_link: geometry collision mesh filename=../../meshes/bumi3/waist_yaw_link.STL; visual mesh filename=../../meshes/bumi3/waist_yaw_link.STL
