Commit message: add_bumi3_stl.urdf

File: gear_sonic/data/assets/robot_description/urdf/bumi3/bumi3_stl.urdf (robot description, URDF)
Before this commit: robot BUMI_V3.0_260119, 22 links, 21 joints
Links:
- link base_link: geometry collision mesh filename=../../meshes/bumi3/base_link.STL; visual mesh filename=../../meshes/bumi3/base_link.STL
- link l_ankle_roll_link: geometry collision mesh filename=../../meshes/bumi3/l_ankle_roll_link.STL; visual mesh filename=../../meshes/bumi3/l_ankle_roll_link.STL
- link l_elbow_pitch_link: geometry collision mesh filename=../../meshes/bumi3/l_elbow_pitch_link.STL; visual mesh filename=../../meshes/bumi3/l_elbow_pitch_link.STL
- link l_knee_pitch_link: mass 1.762561e+00 -> 1.529376e+00
- link r_ankle_roll_link: geometry collision mesh filename=../../meshes/bumi3/r_ankle_roll_link.STL; visual mesh filename=../../meshes/bumi3/r_ankle_roll_link.STL
- link r_elbow_pitch_link: geometry collision mesh filename=../../meshes/bumi3/r_elbow_pitch_link.STL; visual mesh filename=../../meshes/bumi3/r_elbow_pitch_link.STL
- link r_knee_pitch_link: mass 1.762561e+00 -> 1.529376e+00
Joints:
- joint l_arm_roll_joint: limit lower=-1.04 upper=1.4 effort=0 velocity=0 -> lower=-0.14 upper=1.94 effort=0 velocity=0
- joint r_arm_roll_joint: limit lower=-1.4 upper=1.04 effort=0 velocity=0 -> lower=-1.94 upper=0.14 effort=0 velocity=0
